Commit message: Fix robot stability with caster wheels

File: urdf/tunnel_robot.urdf.xacro (robot description, xacro)
@@ -1,10 +1,9 @@
 <?xml version="1.0"?>
 <robot xmlns:xacro="http://www.ros.org/wiki/xacro" name="tunnel_robot">
-  <!-- Base Link -->
   <link name="base_footprint"/>
   <joint name="base_joint" type="fixed">
     <parent link="base_footprint"/>
     <child link="base_link"/>
-    <origin xyz="0 0 0.1" rpy="0 0 0"/>
+    <origin xyz="0 0 0.15" rpy="0 0 0"/>
   </joint>
   <link name="base_link">
@@ -31,5 +30,5 @@
     <parent link="base_link"/>
     <child link="left_wheel"/>
-    <origin xyz="0 0.22 -0.05" rpy="-1.5708 0 0"/>
+    <origin xyz="0 0.225 -0.1" rpy="-1.5708 0 0"/>
     <axis xyz="0 0 1"/>
   </joint>
@@ -57,5 +56,5 @@
     <parent link="base_link"/>
     <child link="right_wheel"/>
-    <origin xyz="0 -0.22 -0.05" rpy="-1.5708 0 0"/>
+    <origin xyz="0 -0.225 -0.1" rpy="-1.5708 0 0"/>
     <axis xyz="0 0 1"/>
   </joint>
@@ -77,4 +76,50 @@
     </inertial>
   </link>
+  <!-- Front Caster -->
+  <joint name="front_caster_joint" type="fixed">
+    <parent link="base_link"/>
+    <child link="front_caster"/>
+    <origin xyz="0.25 0 -0.15" rpy="0 0 0"/>
+  </joint>
+  <link name="front_caster">
+    <visual>
+      <geometry>
+        <sphere radius="0.05"/>
+      </geometry>
+      <material name="black"/>
+    </visual>
+    <collision>
+      <geometry>
+        <sphere radius="0.05"/>
+      </geometry>
+    </collision>
+    <inertial>
+      <mass value="0.5"/>
+      <inertia ixx="0.001" ixy="0" ixz="0" iyy="0.001" iyz="0" izz="0.001"/>
+    </inertial>
+  </link>
+  <!-- Back Caster -->
+  <joint name="back_caster_joint" type="fixed">
+    <parent link="base_link"/>
+    <child link="back_caster"/>
+    <origin xyz="-0.25 0 -0.15" rpy="0 0 0"/>
+  </joint>
+  <link name="back_caster">
+    <visual>
+      <geometry>
+        <sphere radius="0.05"/>
+      </geometry>
+      <material name="black"/>
+    </visual>
+    <collision>
+      <geometry>
+        <sphere radius="0.05"/>
+      </geometry>
+    </collision>
+    <inertial>
+      <mass value="0.5"/>
+      <inertia ixx="0.001" ixy="0" ixz="0" iyy="0.001" iyz="0" izz="0.001"/>
+    </inertial>
+  </link>
   <!-- IMU Link -->
   <joint name="imu_joint" type="fixed">
@@ -109,10 +154,19 @@
     </visual>
   </link>
-  <!-- Gazebo Differential Drive Plugin -->
+  <!-- Caster friction fix -->
+  <gazebo reference="front_caster">
+    <mu1>0.0</mu1>
+    <mu2>0.0</mu2>
+  </gazebo>
+  <gazebo reference="back_caster">
+    <mu1>0.0</mu1>
+    <mu2>0.0</mu2>
+  </gazebo>
+  <!-- Differential Drive Plugin -->
   <gazebo>
     <plugin name="diff_drive" filename="libgazebo_ros_diff_drive.so">
       <left_joint>left_wheel_joint</left_joint>
       <right_joint>right_wheel_joint</right_joint>
-      <wheel_separation>0.44</wheel_separation>
+      <wheel_separation>0.45</wheel_separation>
       <wheel_diameter>0.2</wheel_diameter>
       <max_wheel_torque>20</max_wheel_torque>
