Commit message: Update ROS2 tunnel inspection project

File: urdf/tunnel_robot.urdf.xacro (robot description, xacro)
@@ -30,5 +30,5 @@
     <parent link="base_link"/>
     <child link="left_wheel"/>
-    <origin xyz="0 0.225 -0.1" rpy="-1.5708 0 0"/>
+    <origin xyz="0 0.225 -0.05" rpy="-1.5708 0 0"/>
     <axis xyz="0 0 1"/>
   </joint>
@@ -56,5 +56,5 @@
     <parent link="base_link"/>
     <child link="right_wheel"/>
-    <origin xyz="0 -0.225 -0.1" rpy="-1.5708 0 0"/>
+    <origin xyz="0 -0.225 -0.05" rpy="-1.5708 0 0"/>
     <axis xyz="0 0 1"/>
   </joint>
@@ -80,5 +80,5 @@
     <parent link="base_link"/>
     <child link="front_caster"/>
-    <origin xyz="0.25 0 -0.15" rpy="0 0 0"/>
+    <origin xyz="0.25 0 -0.10" rpy="0 0 0"/>
   </joint>
   <link name="front_caster">
@@ -103,5 +103,5 @@
     <parent link="base_link"/>
     <child link="back_caster"/>
-    <origin xyz="-0.25 0 -0.15" rpy="0 0 0"/>
+    <origin xyz="-0.25 0 -0.10" rpy="0 0 0"/>
   </joint>
   <link name="back_caster">
@@ -190,5 +190,5 @@
             <noise type="gaussian">
               <mean>0.0</mean>
-              <stddev>0.01</stddev>
+              <stddev>0.0</stddev>
             </noise>
           </x>
@@ -196,5 +196,5 @@
             <noise type="gaussian">
               <mean>0.0</mean>
-              <stddev>0.01</stddev>
+              <stddev>0.0</stddev>
             </noise>
           </y>
@@ -202,5 +202,5 @@
             <noise type="gaussian">
               <mean>0.0</mean>
-              <stddev>0.01</stddev>
+              <stddev>0.0</stddev>
             </noise>
           </z>
@@ -210,5 +210,5 @@
             <noise type="gaussian">
               <mean>0.0</mean>
-              <stddev>0.1</stddev>
+              <stddev>0.0</stddev>
             </noise>
           </x>
@@ -216,5 +216,5 @@
             <noise type="gaussian">
               <mean>0.0</mean>
-              <stddev>0.1</stddev>
+              <stddev>0.0</stddev>
             </noise>
           </y>
@@ -222,5 +222,5 @@
             <noise type="gaussian">
               <mean>0.0</mean>
-              <stddev>0.1</stddev>
+              <stddev>0.0</stddev>
             </noise>
           </z>
@@ -231,8 +231,8 @@
           <remapping>~/out:=imu/data</remapping>
         </ros>
-        <initial_orientation_as_reference>false</initial_orientation_as_reference>
+        <initial_orientation_as_reference>true</initial_orientation_as_reference>
         <frame_name>imu_link</frame_name>
         <update_rate>100</update_rate>
-        <gaussian_noise>0.01</gaussian_noise>
+        <gaussian_noise>0.0</gaussian_noise>
       </plugin>
     </sensor>
